Commit message: overworked description

File: mp_description/urdf/mp_description.urdf.xacro (robot description, xacro)
@@ -1,177 +1,134 @@
 <?xml version="1.0"?>
-<robot xmlns:xacro="http://www.ros.org/wiki/xacro" name="mecanum_robot">
-  <!-- ================================================== -->
-  <!-- Parameters -->
-  <!-- ================================================== -->
-  <xacro:property name="wheel_radius" value="0.09"/>
-  <xacro:property name="wheel_width" value="0.04"/>
-  <!-- Front–rear distance -->
-  <xacro:property name="wheelbase" value="0.103"/>
-  <!-- Left–right distance -->
-  <xacro:property name="wheel_distance" value="0.18"/>
-  <xacro:property name="chassis_length" value="0.45"/>
-  <xacro:property name="chassis_width"  value="0.35"/>
-  <xacro:property name="chassis_height" value="0.08"/>
-  <!-- ================================================== -->
-  <!-- Base Link -->
-  <!-- ================================================== -->
+<!--
+  Robot: mecanum_robot
+  Generated by: LinkForge v1.2.3
+  https://github.com/arounamounchili/linkforge
+  Date: 2026-02-28 18:07:18
+-->
+<robot name="mecanum_robot">
+  <!-- Links -->
   <link name="base_link">
     <visual>
+      <origin xyz="0 0 -0.000069" rpy="0 0 0" />
       <geometry>
-        <mesh filename="package://mp_description/meshes/platform.stl" />
+        <mesh filename="meshes\base_link_visual.obj" />
       </geometry>
-      <origin xyz="0 0 ${chassis_height/2}"/>
     </visual>
     <collision>
+      <origin xyz="0 0 -0.000069" rpy="0 0 0" />
       <geometry>
-        <mesh filename="package://mp_description/meshes/platform_c.stl" />
+        <box size="0.259997 0.179998 0.077499" />
       </geometry>
-      <origin xyz="0 0 ${chassis_height/2}"/>
     </collision>
     <inertial>
-      <mass value="10.0"/>
-      <origin xyz="0 0 ${chassis_height/2}"/>
-      <inertia ixx="0.2" iyy="0.2" izz="0.2"
-               ixy="0" ixz="0" iyz="0"/>
+      <mass value="5" />
+      <inertia ixx="0.016002" ixy="0" ixz="0" iyy="0.030668" iyz="0" izz="0.041666" />
     </inertial>
   </link>
-  <!-- ================================================== -->
-  <!-- Wheel Macro -->
-  <!-- ================================================== -->
-  <xacro:macro name="mecanum_wheel" params="name x y">
-    <link name="${name}_link">
-      <visual>
-        <geometry>
-          <mesh filename="package://mp_description/meshes/wheel.stl" />
-          <!-- <cylinder radius="${wheel_radius}" length="${wheel_width}"/> -->
-        </geometry>
-        <origin rpy="1.5708 0 0"/>
-      </visual>
-      <collision>
-        <geometry>
-          <cylinder radius="${wheel_radius}" length="${wheel_width}"/>
-        </geometry>
-        <origin rpy="1.5708 0 0"/>
-      </collision>
-      <inertial>
-        <mass value="1.0"/>
-        <inertia ixx="0.001" iyy="0.001" izz="0.001"
-                 ixy="0" ixz="0" iyz="0"/>
-      </inertial>
-    </link>
-    <joint name="${name}_joint" type="continuous">
-      <parent link="base_link"/>
-      <child link="${name}_link"/>
-      <origin xyz="${x} ${y} ${wheel_radius}"/>
-      <axis xyz="0 1 0"/>
-    </joint>
-  </xacro:macro>
-  <!-- ================================================== -->
-  <!-- Wheel Instances -->
-  <!-- ================================================== -->
-  <xacro:mecanum_wheel
-    name="front_left"
-    x="${ wheelbase/2 }"
-    y="${ wheel_distance/2 }"/>
-  <xacro:mecanum_wheel
-    name="front_right"
-    x="${ wheelbase/2 }"
-    y="${-wheel_distance/2 }"/>
-  <xacro:mecanum_wheel
-    name="rear_left"
-    x="${-wheelbase/2 }"
-    y="${ wheel_distance/2 }"/>
-  <xacro:mecanum_wheel
-    name="rear_right"
-    x="${-wheelbase/2 }"
-    y="${-wheel_distance/2 }"/>
-  <!-- ================================================== -->
-  <!-- ros2_control (Custom Hardware Interface) -->
-  <!-- ================================================== -->
-  <!-- <ros2_control name="mecanum_base_mock" type="system">
-    <hardware>
-      <plugin>mock_components/GenericSystem</plugin>
-      <param name="update_rate">100.0</param>
-    </hardware>
-    <joint name="front_left_joint">
-      <command_interface name="velocity"/>
-      <state_interface name="position">
-        <param name="initial_value">0.0</param>
-      </state_interface>
-      <state_interface name="velocity"/>
-    </joint>
-    <joint name="front_right_joint">
-      <command_interface name="velocity"/>
-      <state_interface name="position">
-        <param name="initial_value">0.0</param>
-      </state_interface>
-      <state_interface name="velocity"/>
-    </joint>
-    <joint name="rear_left_joint">
-      <command_interface name="velocity"/>
-      <state_interface name="position">
-        <param name="initial_value">0.0</param>
-      </state_interface>
-      <state_interface name="velocity"/>
-    </joint>
-    <joint name="rear_right_joint">
-      <command_interface name="velocity"/>
-      <state_interface name="position">
-        <param name="initial_value">0.0</param>
-      </state_interface>
-      <state_interface name="velocity"/>
-    </joint>
-  </ros2_control> -->
-  <ros2_control name="mecanum_base" type="system">
-    <hardware>
-      <plugin>robot_interface_test/Robot7DoF</plugin>
-      <param name="serial_dev_name">/dev/ttyUSB1</param>
-      <param name="serial_baud_rate">115200</param>
-      <param name="testParam">0</param>
-    </hardware>
-    <joint name="front_left_joint">
-      <param name="motor_id"> 5 </param>
-      <command_interface name="velocity">
-        <param name="min">-20.0</param>
-        <param name="max">20.0</param>
-      </command_interface>
-      <state_interface name="position">
-        <param name="initial_value">0.0</param>
-      </state_interface>
-      <state_interface name="velocity"/>
-    </joint>
-    <joint name="front_right_joint">
-    <param name="motor_id"> 0 </param>
-      <command_interface name="velocity">
-        <param name="min">-20.0</param>
-        <param name="max">20.0</param>
-      </command_interface>
-      <state_interface name="position">
-        <param name="initial_value">0.0</param>
-      </state_interface>
-      <state_interface name="velocity"/>
-    </joint>
-    <joint name="rear_left_joint">
-    <param name="motor_id"> 2 </param>
-      <command_interface name="velocity">
-        <param name="min">-20.0</param>
-        <param name="max">20.0</param>
-      </command_interface>
-      <state_interface name="position">
-        <param name="initial_value">0.0</param>
-      </state_interface>
-      <state_interface name="velocity"/>
-    </joint>
-    <joint name="rear_right_joint">
-    <param name="motor_id"> 1 </param>
-      <command_interface name="velocity">
-        <param name="min">-20.0</param>
-        <param name="max">20.0</param>
-      </command_interface>
-      <state_interface name="position">
-        <param name="initial_value">0.0</param>
-      </state_interface>
-      <state_interface name="velocity"/>
-    </joint>
-  </ros2_control>
+  <link name="rear_left_wheel">
+    <visual>
+      <origin xyz="0 0 0" rpy="0 0 0" />
+      <geometry>
+        <mesh filename="meshes\rear_left_wheel_visual.obj" />
+      </geometry>
+    </visual>
+    <inertial>
+      <mass value="1" />
+      <inertia ixx="0.000688" ixy="0" ixz="0" iyy="0.000688" iyz="0" izz="0.000998" />
+    </inertial>
+  </link>
+  <link name="front_left_wheel">
+    <visual>
+      <origin xyz="0 0 0" rpy="0 0 0" />
+      <geometry>
+        <mesh filename="meshes\front_left_wheel_visual.obj" />
+      </geometry>
+    </visual>
+    <inertial>
+      <mass value="1" />
+      <inertia ixx="0.000688" ixy="0" ixz="0" iyy="0.000688" iyz="0" izz="0.000998" />
+    </inertial>
+  </link>
+  <link name="rear_right_wheel">
+    <visual>
+      <origin xyz="0 0 0" rpy="0 0 0" />
+      <geometry>
+        <mesh filename="meshes\rear_right_wheel_visual.obj" />
+      </geometry>
+    </visual>
+    <inertial>
+      <mass value="1" />
+      <inertia ixx="0.000688" ixy="0" ixz="0" iyy="0.000688" iyz="0" izz="0.000998" />
+    </inertial>
+  </link>
+  <link name="front_right_wheel">
+    <visual>
+      <origin xyz="0 0 0" rpy="0 0 0" />
+      <geometry>
+        <mesh filename="meshes\front_right_wheel_visual.obj" />
+      </geometry>
+    </visual>
+    <inertial>
+      <mass value="1" />
+      <inertia ixx="0.000688" ixy="0" ixz="0" iyy="0.000688" iyz="0" izz="0.000998" />
+    </inertial>
+  </link>
+  <link name="base_footprint">
+    <inertial>
+      <mass value="1" />
+      <inertia ixx="1" ixy="0" ixz="0" iyy="1" iyz="0" izz="1" />
+    </inertial>
+  </link>
+  <link name="laser">
+    <inertial>
+      <mass value="1" />
+      <inertia ixx="1" ixy="0" ixz="0" iyy="1" iyz="0" izz="1" />
+    </inertial>
+  </link>
+  <link name="camera">
+    <inertial>
+      <mass value="1" />
+      <inertia ixx="1" ixy="0" ixz="0" iyy="1" iyz="0" izz="1" />
+    </inertial>
+  </link>
+  <!-- Joints -->
+  <joint name="front_right_joint" type="continuous">
+    <origin xyz="0.09 -0.071496 0.000175" rpy="1.570796 0 -3.141593" />
+    <parent link="base_link" />
+    <child link="front_right_wheel" />
+    <axis xyz="0 0 1" />
+  </joint>
+  <joint name="rear_right_joint" type="continuous">
+    <origin xyz="-0.09 -0.071496 0.000175" rpy="1.570796 0 -3.141593" />
+    <parent link="base_link" />
+    <child link="rear_right_wheel" />
+    <axis xyz="0 0 1" />
+  </joint>
+  <joint name="front_left_joint" type="continuous">
+    <origin xyz="0.09 0.071504 0.000175" rpy="1.570796 0 0" />
+    <parent link="base_link" />
+    <child link="front_left_wheel" />
+    <axis xyz="0 0 1" />
+  </joint>
+  <joint name="rear_left_joint" type="continuous">
+    <origin xyz="-0.09 0.071504 0.000175" rpy="1.570796 0 0" />
+    <parent link="base_link" />
+    <child link="rear_left_wheel" />
+    <axis xyz="0 0 1" />
+  </joint>
+  <joint name="base_footprint_joint" type="fixed">
+    <origin xyz="0 0 -0.038825" rpy="0 0 0" />
+    <parent link="base_link" />
+    <child link="base_footprint" />
+  </joint>
+  <joint name="laser_joint" type="fixed">
+    <origin xyz="0.070733 0 0.086997" rpy="0 0 -1.570796" />
+    <parent link="base_link" />
+    <child link="laser" />
+  </joint>
+  <joint name="camera_joint" type="fixed">
+    <origin xyz="0.081656 0.036685 0.067712" rpy="-1.570796 0 -1.570796" />
+    <parent link="base_link" />
+    <child link="camera" />
+  </joint>
 </robot>

Commit message: changed mesh location

File: mp_description/urdf/mp_description.urdf.xacro (robot description, xacro)
@@ -12,5 +12,5 @@
       <origin xyz="0 0 -0.000069" rpy="0 0 0" />
       <geometry>
-        <mesh filename="meshes\base_link_visual.obj" />
+        <mesh filename="package://mp_description/meshes/base_link_visual.obj" />
       </geometry>
     </visual>
@@ -30,5 +30,5 @@
       <origin xyz="0 0 0" rpy="0 0 0" />
       <geometry>
-        <mesh filename="meshes\rear_left_wheel_visual.obj" />
+        <mesh filename="package://mp_description/meshes/rear_left_wheel_visual.obj" />
       </geometry>
     </visual>
@@ -42,5 +42,5 @@
       <origin xyz="0 0 0" rpy="0 0 0" />
       <geometry>
-        <mesh filename="meshes\front_left_wheel_visual.obj" />
+        <mesh filename="package://mp_description/meshes/front_left_wheel_visual.obj" />
       </geometry>
     </visual>
@@ -54,5 +54,5 @@
       <origin xyz="0 0 0" rpy="0 0 0" />
       <geometry>
-        <mesh filename="meshes\rear_right_wheel_visual.obj" />
+        <mesh filename="package://mp_description/meshes/rear_right_wheel_visual.obj" />
       </geometry>
     </visual>
@@ -66,5 +66,5 @@
       <origin xyz="0 0 0" rpy="0 0 0" />
       <geometry>
-        <mesh filename="meshes\front_right_wheel_visual.obj" />
+        <mesh filename="package://mp_description/meshes/front_right_wheel_visual.obj" />
       </geometry>
     </visual>

File: mp_description/urdf/test.urdf (robot description, URDF)
Before this commit: robot mecanum_robot, 5 links, 4 joints
Links:
- removed link front_left_link
- removed link front_right_link
- removed link rear_left_link
- removed link rear_right_link
- added link base_footprint, mass 1
- added link camera, mass 1
- added link front_left_wheel, mass 1; visual mesh filename=meshes\front_left_wheel_visual.obj
- added link front_right_wheel, mass 1; visual mesh filename=meshes\front_right_wheel_visual.obj
- added link laser, mass 1
- added link rear_left_wheel, mass 1; visual mesh filename=meshes\rear_left_wheel_visual.obj
- added link rear_right_wheel, mass 1; visual mesh filename=meshes\rear_right_wheel_visual.obj
- link base_link: mass 10.0 -> 5; geometry collision box size=0.259997 0.179998 0.077499; visual mesh filename=meshes\base_link_visual.obj
Joints:
- added joint base_footprint_joint: type fixed, parent base_link, child base_footprint, origin xyz=0 0 -0.038825 rpy=0 0 0
- added joint camera_joint: type fixed, parent base_link, child camera, origin xyz=0.081656 0.036685 0.067712 rpy=-1.570796 0 -1.570796
- added joint laser_joint: type fixed, parent base_link, child laser, origin xyz=0.070733 0 0.086997 rpy=0 0 -1.570796
- joint front_left_joint: axis 0 1 0 -> 0 0 1; child front_left_link -> front_left_wheel; origin xyz=0.2 0.15 0.05 -> xyz=0.09 0.071504 0.000175 rpy=1.570796 0 0
- joint front_right_joint: axis 0 1 0 -> 0 0 1; child front_right_link -> front_right_wheel; origin xyz=0.2 -0.15 0.05 -> xyz=0.09 -0.071496 0.000175 rpy=1.570796 0 -3.141593
- joint rear_left_joint: axis 0 1 0 -> 0 0 1; child rear_left_link -> rear_left_wheel; origin xyz=-0.2 0.15 0.05 -> xyz=-0.09 0.071504 0.000175 rpy=1.570796 0 0
- joint rear_right_joint: axis 0 1 0 -> 0 0 1; child rear_right_link -> rear_right_wheel; origin xyz=-0.2 -0.15 0.05 -> xyz=-0.09 -0.071496 0.000175 rpy=1.570796 0 -3.141593
