Commit message: reworked description

File: mp_description/urdf/mp_description.urdf.xacro (robot description, xacro)
@@ -1,12 +1,20 @@
 <?xml version="1.0"?>
-<!--
-  Robot: mecanum_robot
-  Generated by: LinkForge v1.2.3
-  https://github.com/arounamounchili/linkforge
-  Date: 2026-02-28 18:07:18
--->
-<robot name="mecanum_robot">
-  <!-- Links -->
-  <link name="base_link">
+<robot xmlns:xacro="http://www.ros.org/wiki/xacro" name="mecanum_robot">
+  <!-- ================================================== -->
+  <!-- Parameters -->
+  <!-- ================================================== -->
+  <xacro:property name="wheel_radius" value="0.09"/>
+  <xacro:property name="wheel_width" value="0.04"/>
+  <!-- Front–rear distance -->
+  <xacro:property name="wheelbase" value="0.103"/>
+  <!-- Left–right distance -->
+  <xacro:property name="wheel_distance" value="0.18"/>
+  <xacro:property name="chassis_length" value="0.45"/>
+  <xacro:property name="chassis_width"  value="0.35"/>
+  <xacro:property name="chassis_height" value="0.08"/>
+  <!-- ================================================== -->
+  <!-- Base Link -->
+  <!-- ================================================== -->
+<link name="base_link">
     <visual>
       <origin xyz="0 0 -0.000069" rpy="0 0 0" />
@@ -16,14 +24,15 @@
     </visual>
     <collision>
-      <origin xyz="0 0 -0.000069" rpy="0 0 0" />
-      <geometry>
-        <box size="0.259997 0.179998 0.077499" />
+      <origin xyz="0 0 0" rpy="0 0 0" />
+      <geometry>
+        <box size="0.26 0.18 0.0775" />
       </geometry>
     </collision>
     <inertial>
       <mass value="5" />
-      <inertia ixx="0.016002" ixy="0" ixz="0" iyy="0.030668" iyz="0" izz="0.041666" />
-    </inertial>
-  </link>
+      <inertia ixx="0.016" ixy="0" ixz="0" iyy="0.030668" iyz="0" izz="0.041666" />
+    </inertial>
+  </link>
+  <!-- Rear Left Wheel -->
   <link name="rear_left_wheel">
     <visual>
@@ -38,4 +47,30 @@
     </inertial>
   </link>
+  <joint name="front_left_joint" type="continuous">
+    <origin xyz="0.09 0.071504 0.000175" rpy="1.570796 0 0" />
+    <parent link="base_link" />
+    <child link="front_left_wheel" />
+    <axis xyz="0 0 1" />
+  </joint>
+   <!-- Rear Right Wheel -->
+  <link name="rear_right_wheel">
+    <visual>
+      <origin xyz="0 0 0" rpy="0 0 0" />
+      <geometry>
+        <mesh filename="package://mp_description/meshes/rear_right_wheel_visual.obj" />
+      </geometry>
+    </visual>
+    <inertial>
+      <mass value="1" />
+      <inertia ixx="0.000688" ixy="0" ixz="0" iyy="0.000688" iyz="0" izz="0.000998" />
+    </inertial>
+  </link>
+  <joint name="rear_right_joint" type="continuous">
+    <origin xyz="-0.09 -0.071496 0.000175" rpy="1.570796 0 -3.141593" />
+    <parent link="base_link" />
+    <child link="rear_right_wheel" />
+    <axis xyz="0 0 1" />
+  </joint>
+  <!-- Front Left Wheel -->
   <link name="front_left_wheel">
     <visual>
@@ -50,16 +85,11 @@
     </inertial>
   </link>
-  <link name="rear_right_wheel">
-    <visual>
-      <origin xyz="0 0 0" rpy="0 0 0" />
-      <geometry>
-        <mesh filename="package://mp_description/meshes/rear_right_wheel_visual.obj" />
-      </geometry>
-    </visual>
-    <inertial>
-      <mass value="1" />
-      <inertia ixx="0.000688" ixy="0" ixz="0" iyy="0.000688" iyz="0" izz="0.000998" />
-    </inertial>
-  </link>
+  <joint name="rear_left_joint" type="continuous">
+    <origin xyz="-0.09 0.071504 0.000175" rpy="1.570796 0 0" />
+    <parent link="base_link" />
+    <child link="rear_left_wheel" />
+    <axis xyz="0 0 1" />
+  </joint>
+  <!-- Front Right Wheel -->
   <link name="front_right_wheel">
     <visual>
@@ -74,23 +104,4 @@
     </inertial>
   </link>
-  <link name="base_footprint">
-    <inertial>
-      <mass value="1" />
-      <inertia ixx="1" ixy="0" ixz="0" iyy="1" iyz="0" izz="1" />
-    </inertial>
-  </link>
-  <link name="laser">
-    <inertial>
-      <mass value="1" />
-      <inertia ixx="1" ixy="0" ixz="0" iyy="1" iyz="0" izz="1" />
-    </inertial>
-  </link>
-  <link name="camera">
-    <inertial>
-      <mass value="1" />
-      <inertia ixx="1" ixy="0" ixz="0" iyy="1" iyz="0" izz="1" />
-    </inertial>
-  </link>
-  <!-- Joints -->
   <joint name="front_right_joint" type="continuous">
     <origin xyz="0.09 -0.071496 0.000175" rpy="1.570796 0 -3.141593" />
@@ -99,22 +110,10 @@
     <axis xyz="0 0 1" />
   </joint>
-  <joint name="rear_right_joint" type="continuous">
-    <origin xyz="-0.09 -0.071496 0.000175" rpy="1.570796 0 -3.141593" />
-    <parent link="base_link" />
-    <child link="rear_right_wheel" />
-    <axis xyz="0 0 1" />
-  </joint>
-  <joint name="front_left_joint" type="continuous">
-    <origin xyz="0.09 0.071504 0.000175" rpy="1.570796 0 0" />
-    <parent link="base_link" />
-    <child link="front_left_wheel" />
-    <axis xyz="0 0 1" />
-  </joint>
-  <joint name="rear_left_joint" type="continuous">
-    <origin xyz="-0.09 0.071504 0.000175" rpy="1.570796 0 0" />
-    <parent link="base_link" />
-    <child link="rear_left_wheel" />
-    <axis xyz="0 0 1" />
-  </joint>
+  <link name="base_footprint">
+    <inertial>
+      <mass value="1" />
+      <inertia ixx="1" ixy="0" ixz="0" iyy="1" iyz="0" izz="1" />
+    </inertial>
+  </link>
   <joint name="base_footprint_joint" type="fixed">
     <origin xyz="0 0 -0.038825" rpy="0 0 0" />
@@ -122,4 +121,10 @@
     <child link="base_footprint" />
   </joint>
+  <link name="laser">
+    <inertial>
+      <mass value="1" />
+      <inertia ixx="1" ixy="0" ixz="0" iyy="1" iyz="0" izz="1" />
+    </inertial>
+  </link>
   <joint name="laser_joint" type="fixed">
     <origin xyz="0.070733 0 0.086997" rpy="0 0 -1.570796" />
@@ -127,4 +132,10 @@
     <child link="laser" />
   </joint>
+  <link name="camera">
+    <inertial>
+      <mass value="1" />
+      <inertia ixx="1" ixy="0" ixz="0" iyy="1" iyz="0" izz="1" />
+    </inertial>
+  </link>
   <joint name="camera_joint" type="fixed">
     <origin xyz="0.081656 0.036685 0.067712" rpy="-1.570796 0 -1.570796" />
@@ -132,3 +143,145 @@
     <child link="camera" />
   </joint>
+  <!-- ================================================== -->
+  <!-- Wheel Macro -->
+  <!-- ================================================== -->
+  <!--
+  <xacro:macro name="mecanum_wheel" params="name x y">
+    <link name="${name}_link">
+      <visual>
+        <geometry>
+          <mesh filename="package://mp_description/meshes/wheel.stl" />
+        </geometry>
+        <origin rpy="1.5708 0 0"/>
+      </visual>
+      <collision>
+        <geometry>
+          <cylinder radius="${wheel_radius}" length="${wheel_width}"/>
+        </geometry>
+        <origin rpy="1.5708 0 0"/>
+      </collision>
+      <inertial>
+        <mass value="1.0"/>
+        <inertia ixx="0.001" iyy="0.001" izz="0.001"
+                 ixy="0" ixz="0" iyz="0"/>
+      </inertial>
+    </link>
+    <joint name="${name}_joint" type="continuous">
+      <parent link="base_link"/>
+      <child link="${name}_link"/>
+      <origin xyz="${x} ${y} ${wheel_radius}"/>
+      <axis xyz="0 1 0"/>
+    </joint>
+  </xacro:macro>
+  -->
+  <!-- ================================================== -->
+  <!-- Wheel Instances -->
+  <!-- ================================================== -->
+  <!--
+  <xacro:mecanum_wheel
+    name="front_left"
+    x="${ wheelbase/2 }"
+    y="${ wheel_distance/2 }"/>
+  <xacro:mecanum_wheel
+    name="front_right"
+    x="${ wheelbase/2 }"
+    y="${-wheel_distance/2 }"/>
+  <xacro:mecanum_wheel
+    name="rear_left"
+    x="${-wheelbase/2 }"
+    y="${ wheel_distance/2 }"/>
+  <xacro:mecanum_wheel
+    name="rear_right"
+    x="${-wheelbase/2 }"
+    y="${-wheel_distance/2 }"/>
+  -->
+  <!-- ================================================== -->
+  <!-- ros2_control (Custom Hardware Interface) -->
+  <!-- ================================================== -->
+  <!-- <ros2_control name="mecanum_base_mock" type="system">
+    <hardware>
+      <plugin>mock_components/GenericSystem</plugin>
+      <param name="update_rate">100.0</param>
+    </hardware>
+    <joint name="front_left_joint">
+      <command_interface name="velocity"/>
+      <state_interface name="position">
+        <param name="initial_value">0.0</param>
+      </state_interface>
+      <state_interface name="velocity"/>
+    </joint>
+    <joint name="front_right_joint">
+      <command_interface name="velocity"/>
+      <state_interface name="position">
+        <param name="initial_value">0.0</param>
+      </state_interface>
+      <state_interface name="velocity"/>
+    </joint>
+    <joint name="rear_left_joint">
+      <command_interface name="velocity"/>
+      <state_interface name="position">
+        <param name="initial_value">0.0</param>
+      </state_interface>
+      <state_interface name="velocity"/>
+    </joint>
+    <joint name="rear_right_joint">
+      <command_interface name="velocity"/>
+      <state_interface name="position">
+        <param name="initial_value">0.0</param>
+      </state_interface>
+      <state_interface name="velocity"/>
+    </joint>
+  </ros2_control> -->
+  <ros2_control name="mecanum_base" type="system">
+    <hardware>
+      <plugin>robot_interface_test/Robot7DoF</plugin>
+      <param name="serial_dev_name">/dev/ttyUSB1</param>
+      <param name="serial_baud_rate">115200</param>
+      <param name="testParam">0</param>
+    </hardware>
+    <joint name="front_left_joint">
+      <param name="motor_id"> 5 </param>
+      <command_interface name="velocity">
+        <param name="min">-20.0</param>
+        <param name="max">20.0</param>
+      </command_interface>
+      <state_interface name="position">
+        <param name="initial_value">0.0</param>
+      </state_interface>
+      <state_interface name="velocity"/>
+    </joint>
+    <joint name="front_right_joint">
+    <param name="motor_id"> 0 </param>
+      <command_interface name="velocity">
+        <param name="min">-20.0</param>
+        <param name="max">20.0</param>
+      </command_interface>
+      <state_interface name="position">
+        <param name="initial_value">0.0</param>
+      </state_interface>
+      <state_interface name="velocity"/>
+    </joint>
+    <joint name="rear_left_joint">
+    <param name="motor_id"> 2 </param>
+      <command_interface name="velocity">
+        <param name="min">-20.0</param>
+        <param name="max">20.0</param>
+      </command_interface>
+      <state_interface name="position">
+        <param name="initial_value">0.0</param>
+      </state_interface>
+      <state_interface name="velocity"/>
+    </joint>
+    <joint name="rear_right_joint">
+    <param name="motor_id"> 1 </param>
+      <command_interface name="velocity">
+        <param name="min">-20.0</param>
+        <param name="max">20.0</param>
+      </command_interface>
+      <state_interface name="position">
+        <param name="initial_value">0.0</param>
+      </state_interface>
+      <state_interface name="velocity"/>
+    </joint>
+  </ros2_control>
 </robot>

Commit message: changed rootlink to be base_framelink

File: mp_description/urdf/mp_description.urdf.xacro (robot description, xacro)
@@ -16,5 +16,6 @@
   <!-- Base Link -->
   <!-- ================================================== -->
-<link name="base_link">
+  <link name="base_footprint"/>
+  <link name="base_link">
     <visual>
       <origin xyz="0 0 -0.000069" rpy="0 0 0" />
@@ -34,4 +35,9 @@
     </inertial>
   </link>
+  <joint name="base_link_joint" type="fixed">
+    <origin xyz="0 0 0.038825" rpy="0 0 0" />
+    <parent link="base_footprint" />
+    <child link="base_link" />
+  </joint>
   <!-- Rear Left Wheel -->
   <link name="rear_left_wheel">
@@ -109,15 +115,4 @@
     <child link="front_right_wheel" />
     <axis xyz="0 0 1" />
-  </joint>
-  <link name="base_footprint">
-    <inertial>
-      <mass value="1" />
-      <inertia ixx="1" ixy="0" ixz="0" iyy="1" iyz="0" izz="1" />
-    </inertial>
-  </link>
-  <joint name="base_footprint_joint" type="fixed">
-    <origin xyz="0 0 -0.038825" rpy="0 0 0" />
-    <parent link="base_link" />
-    <child link="base_footprint" />
   </joint>
   <link name="laser">
